Commit message: add d435

File: xarm_description/urdf/xarm7/xarm7.urdf.xacro (robot description, xacro)
@@ -261,4 +261,21 @@
         origin_xyz="0 0 0"
         origin_rpy="0 0 0" />
+        <!-- Wire visual cylinder -->
+      <visual name="${prefix}link7_wire_visual">
+        <!-- position/orientation relative to link7 frame -->
+        <origin xyz="0.0 -0.04 -0.014" rpy="1.5708 0 0"/>
+        <geometry>
+          <cylinder radius="0.01" length="0.06"/>
+        </geometry>
+        <material name="${prefix}WireBlack">
+          <color rgba="0.01 0.01 0.01 1.0"/>
+        </material>
+      </visual>
+      <collision name="${prefix}link7_wire_collision">
+        <origin xyz="0.0 -0.04 -0.014" rpy="1.5708 0 0"/>
+        <geometry>
+          <cylinder radius="0.01" length="0.06"/>
+        </geometry>
+      </collision>
     </link>
     <joint name="${prefix}joint7" type="revolute">

File: xarm_description/urdf/xarm_device.urdf (robot description, URDF)
Before this commit: robot UF_ROBOT, 17 links, 16 joints
Links:
- added link camera_color_frame
- added link camera_color_optical_frame
- added link camera_depth_frame
- added link camera_depth_optical_frame
- added link camera_left_ir_frame
- added link camera_left_ir_optical_frame
- added link camera_link
- added link camera_right_ir_frame
- added link camera_right_ir_optical_frame
- added link world
- link left_finger: geometry collision mesh filename=package://meshes/gripper/xarm/left_finger.stl; visual mesh filename=package://meshes/gripper/xarm/left_finger.stl
- link left_inner_knuckle: geometry collision mesh filename=package://meshes/gripper/xarm/left_inner_knuckle.stl; visual mesh filename=package://meshes/gripper/xarm/left_inner_knuckle.stl
- link left_outer_knuckle: geometry collision mesh filename=package://meshes/gripper/xarm/left_outer_knuckle.stl; visual mesh filename=package://meshes/gripper/xarm/left_outer_knuckle.stl
- link link1: geometry collision mesh filename=package://meshes/xarm7/visual/link1.stl; visual mesh filename=package://meshes/xarm7/visual/link1.stl
- link link2: geometry collision mesh filename=package://meshes/xarm7/visual/link2.stl; visual mesh filename=package://meshes/xarm7/visual/link2.stl
- link link3: geometry collision mesh filename=package://meshes/xarm7/visual/link3.stl; visual mesh filename=package://meshes/xarm7/visual/link3.stl
- link link4: geometry collision mesh filename=package://meshes/xarm7/visual/link4.stl; visual mesh filename=package://meshes/xarm7/visual/link4.stl
- link link5: geometry collision mesh filename=package://meshes/xarm7/visual/link5.stl; visual mesh filename=package://meshes/xarm7/visual/link5.stl
- link link6: geometry collision mesh filename=package://meshes/xarm7/visual/link6.stl; visual mesh filename=package://meshes/xarm7/visual/link6.stl
- link link7: geometry collision cylinder length=0.06 radius=0.01; collision mesh filename=package://meshes/end_tool/collision/end_tool.stl
- link link_base: geometry collision mesh filename=package://meshes/xarm7/visual/link_base.stl; visual mesh filename=package://meshes/xarm7/visual/link_base.stl
- link link_eef: geometry collision mesh filename=package://meshes/camera/realsense/collision/d435_with_cam_s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; visual mesh filename=package://meshes/camera/realsense/visual/d435_with_cam_stan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
- link right_finger: geometry collision mesh filename=package://meshes/gripper/xarm/right_finger.stl; visual mesh filename=package://meshes/gripper/xarm/right_finger.stl
- link right_inner_knuckle: geometry collision mesh filename=package://meshes/gripper/xarm/right_inner_knuckle.stl; visual mesh filename=package://meshes/gripper/xarm/right_inner_knuckle.stl
- link right_outer_knuckle: geometry collision mesh filename=package://meshes/gripper/xarm/right_outer_knuckle.stl; visual mesh filename=package://meshes/gripper/xarm/right_outer_knuckle.stl
- link xarm_gripper_base_link: geometry collision mesh filename=package://meshes/gripper/xarm/base_link.stl; visual mesh filename=package://meshes/gripper/xarm/base_link.stl
Joints:
- added joint camera_color_joint: type fixed, parent camera_link, child camera_color_frame, origin xyz=0 0.015 0 rpy=0 0 0
- added joint camera_color_optical_joint: type fixed, parent camera_color_frame, child camera_color_optical_frame, origin xyz=0 0 0 rpy=-1.5707963267948966 0 -1.5707963267948966
- added joint camera_depth_joint: type fixed, parent camera_link, child camera_depth_frame, origin xyz=0 0 0 rpy=0 0 0
- added joint camera_depth_optical_joint: type fixed, parent camera_depth_frame, child camera_depth_optical_frame, origin xyz=0 0 0 rpy=-1.5707963267948966 0 -1.5707963267948966
- added joint camera_left_ir_joint: type fixed, parent camera_link, child camera_left_ir_frame, origin xyz=0 0 0 rpy=0 0 0
- added joint camera_left_ir_optical_joint: type fixed, parent camera_left_ir_frame, child camera_left_ir_optical_frame, origin xyz=0 0 0 rpy=-1.5707963267948966 0 -1.5707963267948966
- added joint camera_link_joint: type fixed, parent link_eef, child camera_link, origin xyz=0.06746 -0.0175 0.0237 rpy=3.141592653589793 -1.5707963267948966 0
- added joint camera_right_ir_joint: type fixed, parent camera_link, child camera_right_ir_frame, origin xyz=0 -0.050 0 rpy=0 0 0
- added joint camera_right_ir_optical_joint: type fixed, parent camera_right_ir_frame, child camera_right_ir_optical_frame, origin xyz=0 0 0 rpy=-1.5707963267948966 0 -1.5707963267948966
- added joint world_joint: type fixed, parent world, child link_base, origin xyz=0 0 0 rpy=0 0 0
- joint joint1: origin xyz=0 0 0.267 rpy=0 0 0 -> xyz=-0.0012024487368762493 7.451373676303774e-05 0.26563310623168945 rpy=-0.0016957371262833476 -0.0025385997723788023 2.1524006115214434e-06
- joint joint2: origin xyz=0 0 0 rpy=-1.5708 0 0 -> xyz=-4.0552084101364017e-05 -0.0003101295733358711 -5.259135491542111e-07 rpy=-1.5691006183624268 0.0025385997723788023 2.1524006115214434e-06
- joint joint3: origin xyz=0 -0.293 0 rpy=1.5708 0 0 -> xyz=-5.514011354534887e-05 -0.29205965995788574 -0.0007868116954341531 rpy=1.5734903812408447 7.152952434807958e-07 -0.0005310137057676911
- joint joint4: origin xyz=0.0525 0 0 rpy=1.5708 0 0 -> xyz=0.05300402641296387 0.0008404537802562118 -1.6123338753004646e-07 rpy=1.5706510543823242 0.0005240050959400833 -0.0049373796209692955
- joint joint5: origin xyz=0.0775 -0.3425 0 rpy=1.5708 0 0 -> xyz=0.07665160298347473 -0.34238240122795105 -6.096140714362264e-05 rpy=1.5709741115570068 0.00494197104126215 0.004464946687221527
- joint joint6: origin xyz=0 0 0 rpy=1.5708 0 0 -> xyz=0.0004058310005348176 -0.003988245967775583 -8.553913357900456e-05 rpy=1.5922448635101318 -0.004453355446457863 -0.0018970094388350844
- joint joint7: origin xyz=0.076 0.097 0 rpy=-1.5708 0 0 -> xyz=0.07695576548576355 0.09614047408103943 -0.0021854545921087265 rpy=-1.5954349040985107 0.0013598224613815546 -0.00018891091167461127

File: xarm_description/urdf/xarm_device_workspace.urdf.xacro (robot description, xacro)
@@ -43,8 +43,8 @@
   <xacro:arg name="table_length" default="1.0"/>
   <xacro:arg name="table_width" default="1.0"/>
-  <xacro:arg name="table_height" default="0.05"/>
+  <xacro:arg name="table_height" default="0.1"/>
   <xacro:arg name="table_x" default="0.5"/>
   <xacro:arg name="table_y" default="0.0"/>
-  <xacro:arg name="table_z" default="-0.025"/>
+  <xacro:arg name="table_z" default="0"/>
   <xacro:arg name="pole_length" default="0.06"/>
   <xacro:arg name="pole_width" default="0.06"/>
